File: RF_SWITCH/RF_SWITCH.kicad_pcb (KiCad board)
At the start: 2 copper layers, 69.1 x 62.7 mm, 31 parts, among them J1 Conn_01x01_Male, J2 Conn_01x01_Male, J3 Conn_01x01_Male, J4 Conn_01x01_Male, J5 5V

Commit message: final
Parts:
- removed R1, R2, R3, R4: 50, Resistor_SMD:R_0805_2012Metric
- added H1: MountingHole, MountingHole:MountingHole_2.1mm, F.Cu at (102.6, 80.8)
- added H2: MountingHole, MountingHole:MountingHole_2.1mm, F.Cu at (166.1, 80.8)
- added H3: MountingHole, MountingHole:MountingHole_2.1mm, F.Cu at (166.1, 137.9)
- added H4: MountingHole, MountingHole:MountingHole_2.1mm, F.Cu at (102.6, 137.9)
- R5: value 330 -> 14k
- R6: value 68 -> 1k
- moved D3 31.1 mm to (121.7, 108.7), turned to 90 degrees
- moved D2 28.0 mm to (121.7, 105.2), turned to -90 degrees
- moved D4 12.5 mm to (118.6, 108.7), turned to 90 degrees
- moved D1 7.10 mm to (118.6, 105.2), turned to -90 degrees
- moved C2 0.09 mm to (151.6, 96.6)
- moved J4 0.07 mm to (102.9, 121.2)
- moved Cox4 0.07 mm to (113.3, 135.4)
- renumbered C4 to C3, C3 to C4, Cox4 to Cox3, Cox3 to Cox4, D4 to D3, D3 to D4, J4 to J3, J3 to J4, L4 to L3, L3 to L4
Connections:
- C1 pad 1: Net-(C1-Pad1) -> Net-(Cox1-Pad1)
- C3 pad 1: Net-(C4-Pad1) -> Net-(C3-Pad1)
- C4 pad 1: Net-(C3-Pad1) -> Net-(Cox4-Pad1)
- Cox2 pad 1: Net-(Cox2-Pad1) -> Net-(C2-Pad1)
- Cox3 pad 1: Net-(Cox4-Pad1) -> Net-(C3-Pad1)
- Cox4 pad 1: Net-(Cox3-Pad1) -> Net-(Cox4-Pad1)
Routing:
- net Net-(C5-Pad1): track 97.0 -> 14.7 mm
- net Net-(C3-Pad2): track 4.32 -> 47.1 mm
- net Net-(C2-Pad2): track 4.32 -> 36.4 mm
- net Net-(C4-Pad2): track 4.32 -> 16.5 mm
- net Earth: track 0.00 -> 11.4 mm, vias 1 -> 11
- net Net-(C2-Pad1): track 2.54 -> 13.2 mm
- net Net-(C3-Pad1): track 2.67 -> 12.4 mm
- net Net-(C1-Pad2): track 4.32 -> 11.8 mm
- net Net-(Cox3-Pad1): track 7.36 -> 0.00 mm
- net Net-(Cox2-Pad1): track 7.36 -> 0.00 mm
- net Net-(Cox1-Pad1): track 7.36 -> 13.5 mm
- net Net-(Cox4-Pad1): track 7.36 -> 12.2 mm
- net Net-(C1-Pad1): track 2.54 -> 0.00 mm
- net Net-(C4-Pad1): track 1.78 -> 0.00 mm
