File: RF_SWITCH/RF_SWITCH.kicad_sch (KiCad schematic)
At the start: 31 parts, among them J1 Conn_01x01_Male, J2 Conn_01x01_Male, J3 Conn_01x01_Male, J4 Conn_01x01_Male, J5 5V

Commit message: final
Parts:
- removed R1, R2, R3, R4: 50, Resistor_SMD:R_0805_2012Metric, symbol Device:R
- added H1, H2, H3, H4: MountingHole, MountingHole:MountingHole_2.1mm, symbol Mechanical:MountingHole
- R5: value 330 -> 14k
- R6: value 68 -> 1k
- renumbered C4 to C3, C3 to C4, Cox4 to Cox3, Cox3 to Cox4, D4 to D3, D3 to D4, J4 to J3, J3 to J4, L4 to L3, L3 to L4
Connections:
- net at Cox2.1 (In): now also C2.1
- net at C1.1: now also Cox1.1 (In)
- net at C4.1: now also Cox4.1 (In)
- net at Cox3.1 (In): now also C3.1
